File: IOT_thing.kicad_sch (KiCad schematic)
At the start: 18 parts, among them J1 USB_C_Receptacle_USB2.0_16P, J2 Conn_01x04, J3 Screw_Terminal_01x03, J4 Screw_Terminal_01x08, J5 Screw_Terminal_01x02, K1 RT314A05, Q1 UMH3N, Q2 UMH3N, Q3 BC817, U1 ESP32-WROOM-32D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

Commit message: Placed all components
Parts:
- added D3: LED_RGBA, symbol Device:LED_RGBA
- added D4: LED, symbol Device:LED
- added H1, H2, H3, H4: Hole_Pad, symbol Mechanical:MountingHole_Pad
- added SW1: SW_SPST, symbol Switch:SW_SPST
- added U6: LM1117MP-3.3, Package_TO_SOT_SMD:SOT-223-3_TabPin2, symbol Regulator_Linear:LM1117MP-3.3
Other:
- moved on the sheet: C1, D1, D2, F1, J2, J3, J4, J5, K1, Q3, U1, U4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
