File: IOT_thing.kicad_sch (KiCad schematic)
At the start: 64 parts, among them J1 USB_C_Receptacle_USB2.0_16P, J2 Conn_01x04, J3 Screw_Terminal_01x03, J4 Screw_Terminal_01x08, J5 Screw_Terminal_01x02, J6 Conn_02x05_Odd_Even, K1 RT314A05, Q1 UMH3N, Q2 UMH3N, Q3 BC817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

Commit message: Finalised the project
Parts:
- U2: footprint Package_TO_SOT_SMD:SOT-666 -> iot-thing_Library_11:SOT-666
- U5: footprint Package_DIP:DIP-22_W7.62mm -> iot-thing_Library_11:DIP-20_W7.62mm
Connections:
- net +3.3V: no longer Q2.1 (E1), Q2.4 (E2), U1.3 (EN)
- net GND: no longer H3.1
- net RX: now also U1.34 (RXD0/IO3); no longer U1.35 (TXD0/IO1)
- net TX: now also U1.35 (TXD0/IO1); no longer U1.34 (RXD0/IO3)
- net at J1.A6 (D+), J1.B6 (D+): now also U2.1 (I/O1); no longer U2.4 (I/O2)
- net at U3.4 (D-): now also U2.4 (I/O2); no longer U2.1 (I/O1)
- net EN: now reaches C15.1, R20.2
- net EN: now also Q2.1 (E1), Q2.4 (E2), U1.3 (EN)
- no-connect marks 28 -> 29
Other:
- moved on the sheet: R20, U2
